File: mercury-1/mercury-1/mercury-1.kicad_sch (KiCad schematic)
At the start: 0 parts

Commit message: Draw.io updated
Other:
- removed sheet 5 Port Ethernet Switch
- removed sheet Arm Subsystem
- removed sheet Nvidia Jetson Orin AGX
- removed sheet Raspberry Pi 4 B
- removed sheet Science Subsystem
- removed sheet Sensors and Serial Multiplexers
- note added: "BILLEE Power/Logic Board"
- note removed: "BILLEE Logic Board"
