File: mercury-1/science.kicad_sch (KiCad schematic)
At the start: 27 parts, among them M11 Pump3, M12 Pump2, M13 Pump1, M14 Linear Actuator, M15 Stirrer, M16 Drill, M17 Drill Module 1, M18 Drill Module 2, M19 Servo 1, M20 Servo 2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

Commit message: Updated Schematic to reflect program
Parts:
- removed M14: Linear Actuator, symbol Motor:Motor_DC
- removed M16: Drill, symbol Motor:Motor_DC
- removed U31, U33: HBRIDGE, symbol logic_board:HBRIDGE
- added M23: Drill, symbol Motor:Motor_DC
- added M24: Linear Actuator, symbol Motor:Motor_DC
- added U34, U35: RoboClaw_2x7A, symbol logic_board:RoboClaw_2x7A
Connections:
- net +22.2V_A/S_OUT: now also U34.36 (M_GND), U35.36 (M_GND)
- net GND: now also U34.10 (S2_GND), U34.36 (M_GND), U35.10 (S2_GND), U35.36 (M_GND)
- net at M18.1 (+): now also U34.33 (M2+)
- net at M18.2 (-): now also U34.34 (M2-)
- net at M17.1 (+): now also U34.31 (M1+)
- net at M17.2 (-): now also U34.32 (M1-)
- net Drill_Module1&2_TX: now reaches A1.D16 (D16/TX2)
- net Drill_Module1&2_TX: now also U34.3 (S1), U35.3 (S1)
- net Drill_Module1&2_RX: now reaches A1.D17 (D17/RX2)
- net Drill_Module1&2_RX: now also U34.7 (S2), U35.7 (S2)
- net Drill_LinAct_TX: now reaches A1.D18 (D18/TX1)
- net Drill_LinAct_RX: now reaches A1.D19 (D19/RX1)
- net DrillM1_IN1: no longer names the net of A1.D8
- net DrillM1_IN2: no longer names the net of A1.D9
- net DrillM1_PWM: no longer names the net of A1.D10
- net DrillM2_IN3: no longer names the net of A1.D11
- net DrillM2_IN4: no longer names the net of A1.D12
- net Drill_IN1: no longer names the net of A1.D5
- net Drill_IN2: no longer names the net of A1.D6
- net Drill_PWM: no longer names the net of A1.D7
- net LinAct_IN1: no longer names the net of A1.D2 (D2_INT0)
- net LinAct_IN2: no longer names the net of A1.D3 (D3_INT1)
- net LinAct_PWM: no longer names the net of A1.D4
- new net: M23.1 (+), U35.31 (M1+)
- new net: M23.2 (-), U35.32 (M1-)
- new net: M24.1 (+), U35.33 (M2+)
- new net: M24.2 (-), U35.34 (M2-)
- no-connect marks 90 -> 151
Other:
- note added: "Drill Modules, Drill and Cache"
- note added: "Power"
- note removed: "Drill, Drill Module and Linear Actuator Control"
- moved on the sheet: A1, D1, M11, M12, M13, M15, M17, M18, M19, M20, M21, M22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
